File: HARDWARE/SOMOS_KICAD/SHIELD_Tiny/SHIELD_Tiny.kicad_pcb (KiCad board)
At the start: 2 copper layers, 40 x 50 mm, 42 parts, among them CN4 MicroUSB, J1 Conn_01x03_Female, J2 Conn_01x06_Female, J3 Conn_01x05_Male, J4 Conn_01x08_Male, T1 MMUN2133LT1G, U1 TPS61090RSAR, U2 MCP73871, U4 RN4871-V_RM118, U5 Tiny-FPGA-B2, U6 MCP112, X1 TERM_OUTPUT_1X2

Commit message: merge pretty libraries into one
Parts:
- added REF**: SOMOS_ELECTRODE, SOMOS:SOMOS_ELECTRODE, F.Cu at (189.8, 109.4)
- added REF**: SOMOS_LOGO, SOMOS:SOMOS_LOGO, F.Cu at (150.2, 107.2)
- U5: footprint SOMOS:TinyFPGA-BX_SM -> SOMOS:TinyFPGA-BX_TH; moved to F.Cu
- moved J3 67.8 mm to (162.6, 59.6), turned to 90 degrees
- moved U6 63.2 mm to (180.2, 89.8)
- moved J4 48.4 mm to (149.8, 60.0)
- moved U4 47.9 mm to (138.0, 107.8), turned to 90 degrees
- moved J2 45.8 mm to (174.8, 60.8)
- moved U5 30.4 mm to (149.8, 90.2)
