File: HARDWARE/SOMOS_KICAD/SHIELD_Tiny/SHIELD_Tiny.sch (KiCad schematic (older format))
At the start: 42 parts, among them CN4 MicroUSB, J1 Conn_01x03_Female, J2 Conn_01x06_Female, J3 Conn_01x05_Male, J4 Conn_01x08_Male, T1 MMUN2133LT1G, U1 TPS61090RSAR, U2 MCP73871, U4 RN4871-V_RM118, U5 Tiny-FPGA-B2, U6 MCP112, X1 TERM_OUTPUT_1X2

Commit message: remove step files
Parts:
- added U?: RN4871, RF_Module:Microchip_RN4871, symbol RF_Bluetooth:RN4871
- U4: symbol RN4871-V_RM118:RN4871-V_RM118 -> SHIELD_Tiny-rescue:RN4871-V_RM118-RN4871-V_RM118
- U6: symbol somos_sym_lib:MCP112 -> SHIELD_Tiny-rescue:MCP112-somos_sym_lib
Changed lines of the file:
@@
 $EndComp
 $Comp
-L RN4871-V_RM118:RN4871-V_RM118 U4
+L SHIELD_Tiny-rescue:RN4871-V_RM118-RN4871-V_RM118 U4
 U 1 1 5F838F73
 P 3950 7150
@@
 BT_TX
 $Comp
-L somos_sym_lib:MCP112 U6
+L SHIELD_Tiny-rescue:MCP112-somos_sym_lib U6
 U 1 1 5F8B892E
 P 6250 6850
@@
 Text GLabel 5200 5000 2    50   Input ~ 0
 3V
+$Comp
+L RF_Bluetooth:RN4871 U?
+U 1 1 5FA05F74
+P 1700 5750
+F 0 "U?" H 1700 6531 50  0000 C CNN
+F 1 "RN4871" H 1700 6440 50  0000 C CNN
+F 2 "RF_Module:Microchip_RN4871" H 1700 5050 50  0001 C CNN
+F 3 "http://ww1.microchip.com/downloads/en/DeviceDoc/50002489A.pdf" H 1200 6300 50  0001 C CNN
+	1    1700 5750
+	1    0    0    -1
+$EndComp
 $EndSCHEMATC
